Commit message: my_robot: urdf: xacro: Change robot appearance
Set chassis to Indigo color.
Set Wheels to Red color.

File: my_robot/urdf/my_robot.xacro (robot description, xacro)
@@ -2,4 +2,10 @@
 <robot name="my_robot" xmlns:xacro="http://www.ros.org/wiki/xacro">
   <xacro:include filename="$(find my_robot)/urdf/my_robot.gazebo" />
+  <material name="indigo">
+    <color rgba="0.29 0 0.51 1"/>
+  </material>
+  <material name="red">
+    <color rgba="0.8 0 0 1"/>
+  </material>
   <link name="robot_footprint"></link>
   <joint name="robot_footprint_joint" type="fixed">
@@ -30,4 +36,5 @@
         <box size=".4 .2 .1"/>
       </geometry>
+      <material name="indigo"/>
     </visual>
     <collision name='back_caster_collision'>
@@ -76,4 +83,5 @@
         <cylinder radius="0.1" length="0.05"/>
       </geometry>
+      <material name="red"/>
     </visual>
   </link>
@@ -106,4 +114,5 @@
         <cylinder radius="0.1" length="0.05"/>
       </geometry>
+      <material name="red"/>
     </visual>
   </link>

Commit message: my_robot: urdf: xacro: Change robot width
Part of the project rubric.

File: my_robot/urdf/my_robot.xacro (robot description, xacro)
@@ -28,5 +28,5 @@
       <origin xyz="0 0 0" rpy=" 0 0 0"/>
       <geometry>
-        <box size=".4 .2 .1"/>
+        <box size=".4 .15 .1"/>
       </geometry>
     </collision>
@@ -34,5 +34,5 @@
       <origin xyz="0 0 0" rpy=" 0 0 0"/>
       <geometry>
-        <box size=".4 .2 .1"/>
+        <box size=".4 .15 .1"/>
       </geometry>
       <material name="indigo"/>
@@ -87,5 +87,5 @@
   </link>
   <joint type="continuous" name="right_wheel_hinge">
-    <origin xyz="0 -0.15 0" rpy="0 0 0"/>
+    <origin xyz="0 -0.1 0" rpy="0 0 0"/>
     <child link="right_wheel"/>
     <parent link="chassis"/>
@@ -118,5 +118,5 @@
   </link>
   <joint type="continuous" name="left_wheel_hinge">
-    <origin xyz="0 0.15 0" rpy="0 0 0"/>
+    <origin xyz="0 0.1 0" rpy="0 0 0"/>
     <child link="left_wheel"/>
     <parent link="chassis"/>

Commit message: my_robot: urdf: xacro: Add optical camera link
For a RGB-D camera in URDF file, we need to add an extra link and an
extra joint to the camera link in order to align the camera image in
Gazebo properly with the robot. The parent link of camera_optical_joint
should be properly configured to the original camera link.

File: my_robot/urdf/my_robot.xacro (robot description, xacro)
@@ -153,4 +153,11 @@
     <child link="camera" />
   </joint>
+  <joint name="camera_optical_joint" type="fixed">
+    <origin xyz="0 0 0" rpy="-1.5707 0 -1.5707"/>
+    <parent link="camera"/>
+    <child link="camera_link_optical"/>
+  </joint>
+  <link name="camera_link_optical">
+  </link>
   <link name="hokuyo">
     <inertial>
